Commit message: single lidar push

File: urdf/touch.urdf (robot description, URDF)
Before this commit: robot touch, 3 links, 2 joints
Joints:
- joint lidar1_joint: origin xyz=2.745 -0.1 0.1 rpy=0 0 1.5708 -> xyz=-0.07 -0.035 0.1 rpy=0 0 -1.5708

Commit message: modified real testing

File: urdf/touch.urdf (robot description, URDF)
Before this commit: robot touch, 3 links, 2 joints
Joints:
- joint lidar1_joint: origin xyz=-0.07 -0.035 0.1 rpy=0 0 -1.5708 -> xyz=-0.09 0.725 0.1 rpy=3.1415 0 1.571

Commit message: Update touch.urdf

File: urdf/touch.urdf (robot description, URDF)
Before this commit: robot touch, 3 links, 2 joints
Links:
- removed link lidar2
Joints:
- removed joint lidar2_joint

Commit message: Update touch.urdf

File: urdf/touch.urdf (robot description, URDF)
Before this commit: robot touch, 2 links, 1 joints
Joints:
- joint lidar1_joint: origin xyz=-0.09 0.725 0.1 rpy=3.1415 0 1.571 -> xyz=0.725 -0.09 0.1 rpy=3.1415 0 1.571

Commit message: limited launch file

File: urdf/touch.urdf (robot description, URDF)
Before this commit: robot touch, 2 links, 1 joints
Links:
- removed link lidar1
Joints:
- removed joint lidar1_joint
